File: vscp-din-wireless-esp32-can.kicad_pcb (KiCad board)
At the start: 2 copper layers, 64.8 x 51 mm, 18 parts, among them J1 Conn_Left_I2C, J2 Conn_Right_Power, J3 Conn_01x06, U1 ESP32-WROOM-32D

Commit message: First version gerbers
Parts:
- removed the R8 at (125.2, 92.5)
- added C4: 100nF, Capacitor_SMD:C_0805_2012Metric, F.Cu at (137.4, 88.1)
- added C5: 100nF, Capacitor_SMD:C_0805_2012Metric, F.Cu at (139.2, 79.8)
- added C6: 22pF, Capacitor_SMD:C_0805_2012Metric, F.Cu at (154.4, 72.1)
- added C7: 22pF, Capacitor_SMD:C_0805_2012Metric, F.Cu at (154.4, 88.6)
- added D2: NUP2105L, Package_TO_SOT_SMD:SOT-23, F.Cu at (137.4, 84.8)
- added J4: Conn_01x02, Connector_PinHeader_2.54mm:PinHeader_1x02_P2.54mm_Vertical, F.Cu at (126.0, 85.3)
- added R4: 10K, Resistor_SMD:R_0805_2012Metric, F.Cu at (139.2, 77.2)
- added R9: 120R, Resistor_SMD:R_0805_2012Metric, F.Cu at (129.8, 85.3)
- added U2: MCP2517FD-xSL, Package_SO:SOIC-14_3.9x8.7mm_P1.27mm, F.Cu at (145.5, 76.2)
- added U3: SN65HVD232, Package_SO:SOIC-8_3.9x4.9mm_P1.27mm, F.Cu at (145.3, 85.9)
- added Y1: 4MHz, Crystal:Crystal_SMD_HC49-SD, F.Cu at (154.2, 80.3)
- R7: value 4k7 -> 10K
- moved R7 25.4 mm to (139.2, 72.9), turned to 180 degrees
- moved REF** 3.70 mm to (168.1, 75.2)
- renumbered C4 to C8, R4 to R2, R2 to R6, R6 to R8
Connections:
- net /gpio2 renamed Net-(U1-Pad24)
- net Net-(R1-Pad2) renamed /txcan
- J1 pad 1: /irq -> Net-(J1-Pad1)
- J1 pad 2: /sda -> Net-(D2-Pad2)
- J1 pad 3: /scl -> Net-(D2-Pad1)
- J2 pad 2: Net-(J2-Pad2) -> VCC
- J2 pad 4: VCC -> Net-(J2-Pad4)
- R7 pad 1: /sda -> /irq1
- R8 pad 1: /irq -> /irq0
- U1 pad 11: Net-(U1-Pad11) -> /leda
- U1 pad 12: Net-(U1-Pad12) -> /ledb
- U1 pad 13: Net-(U1-Pad13) -> /SCK
- U1 pad 14: Net-(U1-Pad14) -> /MISO
- U1 pad 16: Net-(U1-Pad16) -> /MOSI
- U1 pad 23: Net-(U1-Pad23) -> /CS
- U1 pad 26: Net-(U1-Pad26) -> /rxcan
- U1 pad 30: /leda -> Net-(U1-Pad30)
- U1 pad 31: /ledb -> Net-(U1-Pad31)
- U1 pad 33: /sda -> Net-(U1-Pad33)
- U1 pad 36: /scl -> Net-(U1-Pad36)
- U1 pad 37: /irq -> Net-(U1-Pad37)
- U1 pad 6: Net-(U1-Pad6) -> /irq1
- U1 pad 7: Net-(U1-Pad7) -> /irq0
Routing:
- net /sda: track 77.1 -> 0.00 mm, vias 1 -> 0
- net /scl: track 77.0 -> 0.00 mm, vias 1 -> 0
- net /irq: track 74.3 -> 0.00 mm, vias 1 -> 0
- net /txcan: track 3.71 -> 58.5 mm
- net /rxcan: track 0.00 -> 53.3 mm, vias 0 -> 2
- net /irq0: track 0.00 -> 51.6 mm, vias 0 -> 4
- net Net-(D2-Pad1): track 0.00 -> 51.4 mm, vias 0 -> 1
- net VCC: track 191.8 -> 239.2 mm
- net Net-(D2-Pad2): track 0.00 -> 40.8 mm
- net /CS: track 0.00 -> 28.9 mm, vias 0 -> 2
- net /irq1: track 0.00 -> 26.7 mm
- net /ledb: track 7.66 -> 29.7 mm, vias 0 -> 1
- net /leda: track 14.8 -> 33.8 mm, vias 0 -> 1
- net Net-(C7-Pad1): track 0.00 -> 18.1 mm
- net /MISO: track 0.00 -> 17.1 mm, vias 0 -> 2
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Other:
- board text added: "VSCP DIN Wireless ESP32 CAN Rev A"
- board text removed: "VSCP DIN Wireless ESP32 M1 Rev A"
